File: FreeCAD/Eprom_USB.kicad_sch (KiCad schematic)
At the start: 91 parts, among them IC1 74HC238, IC2 LM317_TO-220, IC3 Nano V3.1, IC4 LM317_TO-220, IC5 74HC595, IC6 74HC595, IC7 74HC595, J1 24vac, J2 ZIF 40 pins, Q1 BC547, Q10 BC557, Q11 BC547, Q12 BC557, Q2 BC557, Q3 BC547, Q4 BC547, Q5 BC557, Q6 BC557, Q7 BC547, Q8 BC547, Q9 BC557, U1 TL431LP

Commit message: freecad move
Other:
- company: (none) -> ARBIALSOFT
- title: (none) -> Eprom_USB
Changed lines of the file:
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@@
 	(generator_version "9.0")
 	(paper "A2")
+	(title_block
+		(title "Eprom_USB")
+		(company "ARBIALSOFT")
+		(comment 1 "new_hardware")
+	)
 	(junction
 		(at 220.345 261.62)
